Commit message: Added gripper

File: catkin_ws/src/yara_meshes/files/yara.urdf (robot description, URDF)
Before this commit: robot yara, 8 links, 7 joints
Links:
- removed link ee
- removed link link_6
- added link grabbing_point; visual sphere radius=0.0025
- added link left_finger; collision mesh filename=package://yara_meshes/files/left_finger.obj; visual mesh filename=package://yara_meshes/files/left_finger.obj
- added link left_gear; collision mesh filename=package://yara_meshes/files/left_gear.obj; visual mesh filename=package://yara_meshes/files/left_gear.obj
- added link left_hinge; collision mesh filename=package://yara_meshes/files/left_hinge.obj; visual mesh filename=package://yara_meshes/files/left_hinge.obj
- added link palm; collision mesh filename=package://yara_meshes/files/palm.obj; visual mesh filename=package://yara_meshes/files/palm.obj
- added link right_finger; collision mesh filename=package://yara_meshes/files/right_finger.obj; visual mesh filename=package://yara_meshes/files/right_finger.obj
- added link right_gear; collision mesh filename=package://yara_meshes/files/right_gear.obj; visual mesh filename=package://yara_meshes/files/right_gear.obj
- added link right_hinge; collision mesh filename=package://yara_meshes/files/right_hinge.obj; visual mesh filename=package://yara_meshes/files/right_hinge.obj
- added link servo_gear; visual box size=0.001 0.001 0.0005
- link base_link: geometry collision mesh filename=package://yara_meshes/files/base.obj; visual mesh filename=package://yara_meshes/files/base.obj
- link link_1: geometry collision mesh filename=package://yara_meshes/files/Link1.obj; visual mesh filename=package://yara_meshes/files/Link1.obj
- link link_2: geometry collision mesh filename=package://yara_meshes/files/Link2.obj; visual mesh filename=package://yara_meshes/files/Link2.obj
- link link_3: geometry collision mesh filename=package://yara_meshes/files/Link3.obj; visual mesh filename=package://yara_meshes/files/Link3.obj
- link link_4: geometry collision mesh filename=package://yara_meshes/files/Link4.obj; visual mesh filename=package://yara_meshes/files/Link4.obj
- link link_5: geometry collision mesh filename=package://yara_meshes/files/Link5.obj; visual mesh filename=package://yara_meshes/files/Link5.obj
Joints:
- removed joint link_5_to_link_6
- removed joint link_6_to_ee
- added joint left_gear_to_left_finger: type revolute, parent left_gear, child left_finger, origin xyz=-0.022 0 0 rpy=0 0 0, axis 0 0 1, limit lower=-1.5707963267948966 upper=1.5707963267948966 effort=1000.0 velocity=0.5, mimic joint=palm_to_left_gear multiplier=-1
- added joint link_5_to_palm: type revolute, parent link_5, child palm, origin xyz=0 -0.042 0 rpy=0 0 3.141592653589793, axis 0 1 0, limit lower=-1.5707963267948966 upper=1.5707963267948966 effort=1000.0 velocity=0.5
- added joint palm_to_grabbing_point: type fixed, parent palm, child grabbing_point, origin xyz=0 0.08103 0.00156 rpy=0 0 0
- added joint palm_to_left_gear: type revolute, parent palm, child left_gear, origin xyz=-0.014 0.02 0.002 rpy=0 0 0, axis 0 0 1, limit lower=-1.5707963267948966 upper=1.5707963267948966 effort=1000.0 velocity=0.5, mimic joint=palm_to_servo_gear multiplier=-1
- added joint palm_to_left_hinge: type revolute, parent palm, child left_hinge, origin xyz=-0.004 0.042 0.002 rpy=0 0 0, axis 0 0 1, limit lower=-1.5707963267948966 upper=1.5707963267948966 effort=1000.0 velocity=0.5, mimic joint=palm_to_left_gear multiplier=1
- added joint palm_to_right_gear: type revolute, parent palm, child right_gear, origin xyz=0.014 0.02 0.002 rpy=0 0 0, axis 0 0 1, limit lower=-1.5707963267948966 upper=1.5707963267948966 effort=1000.0 velocity=0.5, mimic joint=palm_to_servo_gear multiplier=1
- added joint palm_to_right_hinge: type revolute, parent palm, child right_hinge, origin xyz=0.004 0.042 0.002 rpy=0 0 0, axis 0 0 1, limit lower=-1.5707963267948966 upper=1.5707963267948966 effort=1000.0 velocity=0.5, mimic joint=palm_to_right_gear multiplier=1
- added joint palm_to_servo_gear: type revolute, parent palm, child servo_gear, origin xyz=0 0.0125 0.005 rpy=0 0 0, axis 0 0 1, limit lower=-1.5707963267948966 upper=1.5707963267948966 effort=1000.0 velocity=0.5
- added joint right_gear_to_right_finger: type revolute, parent right_gear, child right_finger, origin xyz=0.022 0 0 rpy=0 0 0, axis 0 0 1, limit lower=-1.5707963267948966 upper=1.5707963267948966 effort=1000.0 velocity=0.5, mimic joint=palm_to_right_gear multiplier=-1
- joint base_to_link_1: limit lower=-1.57079632679 upper=1.57079632679 effort=1000.0 velocity=0.5 -> lower=-1.5707963267948966 upper=1.5707963267948966 effort=1000.0 velocity=0.5; origin xyz=0 0 0.054355 rpy=0 0 0 -> xyz=0 0 0.054 rpy=0 0 3.141592653589793
- joint link_1_to_link_2: axis 1 0 0 -> -1 0 0; limit lower=-1.57079632679 upper=1.57079632679 effort=1000.0 velocity=0.5 -> lower=-1.5707963267948966 upper=1.5707963267948966 effort=1000.0 velocity=0.5; origin xyz=0 .017415 0.055612 rpy=0 0 0 -> xyz=0 -0.017 0.056 rpy=0 0 0
- joint link_2_to_link_3: axis 1 0 0 -> -1 0 0; limit lower=-1.57079632679 upper=1.57079632679 effort=1000.0 velocity=0.5 -> lower=-1.5707963267948966 upper=1.5707963267948966 effort=1000.0 velocity=0.5
- joint link_3_to_link_4: axis 0 1 0 -> 0 -1 0; limit lower=-1.57079632679 upper=1.57079632679 effort=1000.0 velocity=0.5 -> lower=-1.5707963267948966 upper=1.5707963267948966 effort=1000.0 velocity=0.5; origin xyz=0 0.023943 0.043978 rpy=0 0 0 -> xyz=0 -0.024 0.044 rpy=0 0 0
- joint link_4_to_link_5: axis -1 0 0 -> 1 0 0; limit lower=-1.57079632679 upper=1.57079632679 effort=1000.0 velocity=0.5 -> lower=-1.5707963267948966 upper=1.5707963267948966 effort=1000.0 velocity=0.5; origin xyz=0 0.145149 0.003572 rpy=0 0 0 -> xyz=0 -0.146 0.004 rpy=0 0 0
